File: ai03-pcb-guide.kicad_sch (KiCad schematic)
At the start: 24 parts, among them SW1 SW_Push, U1 ATmega32U4-A, Y1 16MHz

Commit message: Part 6 changes
Connections:
- net COL0: now also U1.28 (PB4)
- net COL1: now also U1.27 (PD7)
- net D+: now also R2.1
- net D-: now also R3.1
- net ROW0: now also D1.1 (K), D2.1 (K), U1.26 (PD6)
- net ROW1: now also D3.1 (K), D4.1 (K), U1.29 (PB5)
Changed lines of the file:
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@@
     (stroke (width 0) (type default))
   )
-  (global_label "D-" (shape output) (at 27.94 82.55 0) (fields_autoplaced)
+  (global_label "D-" (shape input) (at 33.02 82.55 180) (fields_autoplaced)
+    (effects (font (size 1.27 1.27)) (justify right))
+    (property "Intersheetrefs" "${INTERSHEET_REFS}" (at 27.2718 82.55 0)
+      (effects (font (size 1.27 1.27)) (justify right) hide)
+    )
+  )
+  (global_label "ROW0" (shape input) (at 113.03 100.33 0) (fields_autoplaced)
     (effects (font (size 1.27 1.27)) (justify left))
-    (property "Intersheetrefs" "${INTERSHEET_REFS}" (at 33.6882 82.55 0)
+    (property "Intersheetrefs" "${INTERSHEET_REFS}" (at 121.1972 100.33 0)
       (effects (font (size 1.27 1.27)) (justify left) hide)
     )
@@
     )
   )
+  (global_label "ROW1" (shape input) (at 113.03 67.31 0) (fields_autoplaced)
+    (effects (font (size 1.27 1.27)) (justify left))
+    (property "Intersheetrefs" "${INTERSHEET_REFS}" (at 121.1972 67.31 0)
+      (effects (font (size 1.27 1.27)) (justify left) hide)
+    )
+  )
   (global_label "COL1" (shape input) (at 204.47 66.04 90) (fields_autoplaced)
     (effects (font (size 1.27 1.27)) (justify left))
     (property "Intersheetrefs" "${INTERSHEET_REFS}" (at 204.47 58.2961 90)
+      (effects (font (size 1.27 1.27)) (justify left) hide)
+    )
+  )
+  (global_label "COL1" (shape input) (at 113.03 102.87 0) (fields_autoplaced)
+    (effects (font (size 1.27 1.27)) (justify left))
+    (property "Intersheetrefs" "${INTERSHEET_REFS}" (at 120.7739 102.87 0)
       (effects (font (size 1.27 1.27)) (justify left) hide)
     )
@@
     )
   )
-  (global_label "ROW0" (shape output) (at 156.21 87.63 0) (fields_autoplaced)
-    (effects (font (size 1.27 1.27)) (justify left))
-    (property "Intersheetrefs" "${INTERSHEET_REFS}" (at 164.3772 87.63 0)
-      (effects (font (size 1.27 1.27)) (justify left) hide)
+  (global_label "ROW0" (shape input) (at 163.83 87.63 180) (fields_autoplaced)
+    (effects (font (size 1.27 1.27)) (justify right))
+    (property "Intersheetrefs" "${INTERSHEET_REFS}" (at 155.6628 87.63 0)
+      (effects (font (size 1.27 1.27)) (justify right) hide)
     )
   )
-  (global_label "ROW1" (shape output) (at 156.21 106.68 0) (fields_autoplaced)
+  (global_label "ROW1" (shape input) (at 163.83 106.68 180) (fields_autoplaced)
+    (effects (font (size 1.27 1.27)) (justify right))
+    (property "Intersheetrefs" "${INTERSHEET_REFS}" (at 155.6628 106.68 0)
+      (effects (font (size 1.27 1.27)) (justify right) hide)
+    )
+  )
+  (global_label "COL0" (shape input) (at 113.03 64.77 0) (fields_autoplaced)
     (effects (font (size 1.27 1.27)) (justify left))
-    (property "Intersheetrefs" "${INTERSHEET_REFS}" (at 164.3772 106.68 0)
+    (property "Intersheetrefs" "${INTERSHEET_REFS}" (at 120.7739 64.77 0)
       (effects (font (size 1.27 1.27)) (justify left) hide)
     )
@@
     )
   )
-  (global_label "D+" (shape output) (at 27.94 80.01 0) (fields_autoplaced)
-    (effects (font (size 1.27 1.27)) (justify left))
-    (property "Intersheetrefs" "${INTERSHEET_REFS}" (at 33.6882 80.01 0)
-      (effects (font (size 1.27 1.27)) (justify left) hide)
+  (global_label "D+" (shape input) (at 33.02 80.01 180) (fields_autoplaced)
+    (effects (font (size 1.27 1.27)) (justify right))
+    (property "Intersheetrefs" "${INTERSHEET_REFS}" (at 27.2718 80.01 0)
+      (effects (font (size 1.27 1.27)) (justify right) hide)
     )
   )
